File: Vadeco-PCB/Vadeco-PCB/Vadeco-PCB.kicad_pcb (KiCad board)
At the start: 2 copper layers, 14 parts, among them J1 Conn_Battery, J2 Conn_TCRT5000, J3 Conn_TCRT5000, J4 Conn_VL53L0X, J5 Conn_VL53L0X, J6 Conn_VL53L0X, J7 Conn_MOTOR_LEFT, J8 Conn_MOTOR_RIGHT, SW1 SW_DIP_x01, U1 Microstart_Remote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

Commit message: final project v1
Parts:
- J1, J2, J3, J4, J5, J6, J7, J8: moved to B.Cu
- moved SW1 177.5 mm to (196.0, 95.0), turned to 90 degrees
- moved J5 172.9 mm to (174.0, 54.0), turned to 270 degrees
- moved A1 154.7 mm to (153.0, 58.0)
- moved U1 148.9 mm to (182.0, 68.0)
- moved J6 133.7 mm to (129.0, 54.0), turned to 270 degrees
- moved J8 130.9 mm to (177.0, 103.0), turned to 180 degrees
- moved U3 127.3 mm to (182.0, 90.0)
- moved J4 118.1 mm to (138.0, 54.0), turned to 270 degrees
- moved U2 118.0 mm to (140.0, 79.0)
- moved J2 113.5 mm to (198.0, 81.0), turned to 180 degrees
- moved J1 106.8 mm to (196.0, 103.0), turned to 90 degrees
- moved J3 91.1 mm to (109.0, 77.0)
- moved U4 60.8 mm to (119.0, 90.0)
- moved J7 43.1 mm to (124.0, 104.0)
Routing:
- net 5V_ARDUINO: track 0.00 -> 177.1 mm, vias 0 -> 7
- net 6V_LM2596: track 0.00 -> 160.0 mm
- net Net-(SW1-Pad2): track 0.00 -> 78.7 mm
- net SDA_VL53L0X: track 0.00 -> 73.3 mm
- net SCL_VL53L0X: track 0.00 -> 71.5 mm, vias 0 -> 3
- net STBY_TB6612FNG: track 0.00 -> 68.7 mm, vias 0 -> 2
- net ANALOG_LINE2: track 0.00 -> 63.1 mm, vias 0 -> 4
- net DISTANCE_03: track 0.00 -> 48.8 mm, vias 0 -> 3
- net SIGNAL_MICROSTART: track 0.00 -> 45.8 mm, vias 0 -> 2
- net PWM_MOTOR_RIGHT: track 0.00 -> 40.1 mm, vias 0 -> 2
- net BIT1_MOTOR_RIGHT: track 0.00 -> 39.6 mm
- net BIT2_MOTOR_LEFT: track 0.00 -> 39.6 mm, vias 0 -> 2
- net BIT2_MOTOR_RIGHT: track 0.00 -> 37.5 mm, vias 0 -> 1
- net DISTANCE_02: track 0.00 -> 35.9 mm, vias 0 -> 3
- net ANALOG_LINE1: track 0.00 -> 35.5 mm
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- added copper zone on B.Cu, net GND
- added copper zone on F.Cu, net GND
Other:
- board outline added: 94 x 54 mm
- board text added: "- ROBOTECH -"
- board text added: "VADECO"

Commit message: generating topside and backside view
Routing:
- net SIGNAL_MICROSTART: vias 2 -> 1

Commit message: schematic v3 and PCB v2
Parts:
- J4, J5, J6: moved to F.Cu
- moved J2 39.9 mm to (165.8, 104.5), turned to 90 degrees
- moved J3 39.7 mm to (137.6, 104.5), turned to 90 degrees
- moved U4 25.3 mm to (144.2, 88.0), turned to 90 degrees
- moved A1 21.9 mm to (139.2, 75.0), turned to 90 degrees
- moved U2 21.5 mm to (119.0, 83.7)
- moved J7 20.5 mm to (144.4, 104.6), turned to 90 degrees
- moved J4 18.8 mm to (156.8, 52.8)
- moved U3 11.1 mm to (171.1, 88.0), turned to 90 degrees
- moved U1 11.1 mm to (192.7, 71.1), turned to 270 degrees
- moved J6 6.49 mm to (135.4, 52.9)
- moved J5 3.40 mm to (177.1, 52.6)
- moved J1 2.72 mm to (193.8, 104.6)
- moved J8 1.48 mm to (176.7, 104.5), turned to 90 degrees
- moved SW1 1.36 mm to (197.1, 95.8), turned to 180 degrees
Connections:
- A1 pad 10: BIT1_MOTOR_RIGHT -> BIT1_MOTOR_LEFT
- A1 pad 11: BIT2_MOTOR_RIGHT -> BIT2_MOTOR_LEFT
- A1 pad 12: STBY_TB6612FNG -> PWM_MOTOR_LEFT
- A1 pad 13: PWM_MOTOR_LEFT -> PWM_MOTOR_RIGHT
- A1 pad 14: PWM_MOTOR_RIGHT -> BIT2_MOTOR_RIGHT
- A1 pad 15: DISTANCE_03 -> BIT1_MOTOR_RIGHT
- A1 pad 5: SIGNAL_MICROSTART -> DISTANCE_03
- A1 pad 8: BIT1_MOTOR_LEFT -> SIGNAL_MICROSTART
- A1 pad 9: BIT2_MOTOR_LEFT -> STBY_TB6612FNG
- J2 pad 1: 5V_ARDUINO -> GND
- J2 pad 2: GND -> 5V_ARDUINO
- J2 pad 3: Net-(J2-Pad3) -> ANALOG_LINE1
- J2 pad 4: ANALOG_LINE1 -> Net-(J2-Pad4)
- J3 pad 1: 5V_ARDUINO -> GND
- J3 pad 2: GND -> 5V_ARDUINO
- J3 pad 3: Net-(J3-Pad3) -> ANALOG_LINE2
- J3 pad 4: ANALOG_LINE2 -> Net-(J3-Pad4)
- J4 pad 1: 5V_ARDUINO -> SDA_VL53L0X
- J4 pad 2: GND -> SCL_VL53L0X
- J4 pad 3: SCL_VL53L0X -> 5V_ARDUINO
- J4 pad 4: SDA_VL53L0X -> GND
- J5 pad 1: 5V_ARDUINO -> DISTANCE_02
- J5 pad 2: GND -> Net-(J5-Pad2)
- J5 pad 3: SCL_VL53L0X -> GND
- J5 pad 5: Net-(J5-Pad5) -> SCL_VL53L0X
- J5 pad 6: DISTANCE_02 -> 5V_ARDUINO
- J6 pad 1: 5V_ARDUINO -> SDA_VL53L0X
- J6 pad 2: GND -> SCL_VL53L0X
- J6 pad 3: SCL_VL53L0X -> 5V_ARDUINO
- J6 pad 4: SDA_VL53L0X -> GND
- U3 pad 6: Net-(J8-Pad1) -> Net-(J8-Pad2)
- U3 pad 7: Net-(J8-Pad2) -> Net-(J8-Pad1)
- U4 pad 4: Net-(J7-Pad1) -> Net-(J7-Pad2)
- U4 pad 5: Net-(J7-Pad2) -> Net-(J7-Pad1)
Routing:
- net GND: track 0.00 -> 49.2 mm
- net STBY_TB6612FNG: track 68.7 -> 31.5 mm, vias 2 -> 0
- net ANALOG_LINE1: track 35.5 -> 70.2 mm, vias 0 -> 3
- net PWM_MOTOR_RIGHT: track 40.1 -> 8.24 mm, vias 2 -> 0
- net BIT1_MOTOR_RIGHT: track 39.6 -> 8.00 mm
- net BIT2_MOTOR_RIGHT: track 37.5 -> 8.12 mm, vias 1 -> 0
- net BIT2_MOTOR_LEFT: track 39.6 -> 16.2 mm, vias 2 -> 0
- net SDA_VL53L0X: track 73.3 -> 51.8 mm
- net SCL_VL53L0X: track 71.5 -> 52.0 mm, vias 3 -> 0
- net DISTANCE_01: track 20.8 -> 40.1 mm, vias 0 -> 1
- net DISTANCE_03: track 48.8 -> 29.9 mm, vias 3 -> 0
- net BIT1_MOTOR_LEFT: track 34.1 -> 16.3 mm, vias 1 -> 0
- net PWM_MOTOR_LEFT: track 31.1 -> 16.1 mm, vias 2 -> 0
- net SIGNAL_MICROSTART: track 45.8 -> 32.3 mm, vias 1 -> 0
- net 5V_ARDUINO: track 177.1 -> 189.5 mm, vias 7 -> 3
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Other:
- board text added: "-ROBOTECH-"
- board text removed: "- ROBOTECH -"
