File: Vadeco-PCB/Vadeco-PCB/Vadeco-PCB.sch (KiCad schematic (older format))
At the start: 12 parts, among them J1 Conn_Battery, J2 Conn_TCRT5000, J3 Conn_TCRT5000, J4 Conn_VL53L0X, J5 Conn_VL53L0X, J6 Conn_VL53L0X, SW1 SW_DIP_x01, U1 Microstart_Remote, U2 LM2596_ADJ, U3 DRIVER_TB6612FNG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

Commit message: schematic done
Parts:
- added J7: Conn_MOTOR_LEFT, symbol Connector_Generic:Conn_01x02
- added J8: Conn_MOTOR_RIGHT, symbol Connector_Generic:Conn_01x02
- U3: value DRIVER_TB6612FNG -> RIGHT_TB6612FNG
- U4: value DRIVER_TB6612FNG -> LEFT_TB6612FNG
Connections:
- net labels added: ANALOG_LINE2, BIT1_MOTOR_LEFT, BIT1_MOTOR_RIGHT, BIT2_MOTOR_LEFT, BIT2_MOTOR_RIGHT, DISTANCE_01, DISTANCE_02, DISTANCE_03, PWM_MOTOR_LEFT, PWM_MOTOR_RIGHT, STBY_TB6612FNG
- net labels removed: DIGITAL_LINE1, LINE_01, LINE_02, LINE_03
- wire segments 2 -> 6
- no-connect marks 13 -> 25
Other:
- moved on the sheet: J1, J2, J3, J4, J5, J6, SW1, U1, U3, U4

Commit message: associating footprint lm2596
Parts:
- U2: footprint (none) -> Converter_DCDC:LM2596_ADJ
Changed lines of the file:
@@
 F 0 "U2" H 6200 3075 50  0000 C CNN
 F 1 "LM2596_ADJ" H 6200 2984 50  0000 C CNN
-F 2 "" H 6150 2750 50  0001 C CNN
+F 2 "Converter_DCDC:LM2596_ADJ" H 6150 2750 50  0001 C CNN
 F 3 "" H 6150 2750 50  0001 C CNN
 	1    6200 2800

Commit message: microstart and tb6612fng footprints
Parts:
- A1: symbol MCU_Module:Arduino_Nano_v3.x -> Vadeco-PCB-rescue:Arduino_Nano_v3.x-MCU_Module
- U1: footprint (none) -> Module:MICROSTART_MODULE
- U2: symbol Regulator_Switching:LM2596_ADJ -> Vadeco-PCB-rescue:LM2596_ADJ-Regulator_Switching
- U4: footprint (none) -> Module:TB6612FNG
Connections:
- no-connect marks 25 -> 26
Changed lines of the file:
@@
 Title "Vadeco"
 Date "2021-05-30"
-Rev "01"
+Rev "02"
 Comp "Robotech"
 Comment1 "Dev.: José Neto"
@@
 $EndDescr
 $Comp
-L MCU_Module:Arduino_Nano_v3.x A1
+L Vadeco-PCB-rescue:Arduino_Nano_v3.x-MCU_Module A1
 U 1 1 60B30CF3
 P 5850 4700
@@
 F 0 "U1" H 2757 5875 50  0000 C CNN
 F 1 "Microstart_Remote" H 2757 5784 50  0000 C CNN
-F 2 "" H 2900 5550 50  0001 C CNN
+F 2 "Module:MICROSTART_MODULE" H 2900 5550 50  0001 C CNN
 F 3 "" H 2900 5550 50  0001 C CNN
 	1    2700 5550
@@
 $EndComp
 $Comp
-L Regulator_Switching:LM2596_ADJ U2
+L Vadeco-PCB-rescue:LM2596_ADJ-Regulator_Switching U2
 U 1 1 60B30F55
 P 6200 2800
@@
 F 0 "U4" H 3200 7475 50  0000 C CNN
 F 1 "LEFT_TB6612FNG" H 3200 7384 50  0000 C CNN
-F 2 "" H 3000 6950 50  0001 C CNN
+F 2 "Module:TB6612FNG" H 3000 6950 50  0001 C CNN
 F 3 "" H 3000 6950 50  0001 C CNN
 	1    3200 6950
@@
 Wire Notes Line style solid
 	7100 2400 7100 3000
+NoConn ~ 5350 5400
 $EndSCHEMATC

Commit message: all footprints associated and placed to PCB
Parts:
- J1, J7, J8: footprint (none) -> Connector_PinHeader_1.00mm:PinHeader_1x02_P1.00mm_Horizontal
- J2, J3: footprint (none) -> Connector_PinHeader_1.00mm:PinHeader_1x04_P1.00mm_Horizontal
- J4, J5, J6: footprint (none) -> Connector_PinHeader_1.00mm:PinHeader_1x06_P1.00mm_Horizontal
- SW1: footprint (none) -> Button_Switch_THT:SW_DIP_SPSTx01_Slide_9.78x4.72mm_W7.62mm_P2.54mm
- U3: footprint (none) -> Module:TB6612FNG
Changed lines of the file:
@@
 F 0 "J1" H 4468 2967 50  0000 C CNN
 F 1 "Conn_Battery" H 4468 2876 50  0000 C CNN
-F 2 "" H 4550 2750 50  0001 C CNN
+F 2 "Connector_PinHeader_1.00mm:PinHeader_1x02_P1.00mm_Horizontal" H 4550 2750 50  0001 C CNN
 F 3 "~" H 4550 2750 50  0001 C CNN
 	1    4550 2750
@@
 F 0 "SW1" H 5300 3017 50  0000 C CNN
 F 1 "SW_DIP_x01" H 5300 2926 50  0000 C CNN
-F 2 "" H 5300 2750 50  0001 C CNN
+F 2 "Button_Switch_THT:SW_DIP_SPSTx01_Slide_9.78x4.72mm_W7.62mm_P2.54mm" H 5300 2750 50  0001 C CNN
 F 3 "~" H 5300 2750 50  0001 C CNN
 	1    5300 2750
@@
 F 0 "J2" H 2568 3917 50  0000 C CNN
 F 1 "Conn_TCRT5000" H 2568 3826 50  0000 C CNN
-F 2 "" H 2650 3600 50  0001 C CNN
+F 2 "Connector_PinHeader_1.00mm:PinHeader_1x04_P1.00mm_Horizontal" H 2650 3600 50  0001 C CNN
 F 3 "~" H 2650 3600 50  0001 C CNN
 	1    2650 3600
@@
 F 0 "J3" H 2568 4567 50  0000 C CNN
 F 1 "Conn_TCRT5000" H 2568 4476 50  0000 C CNN
-F 2 "" H 2650 4250 50  0001 C CNN
+F 2 "Connector_PinHeader_1.00mm:PinHeader_1x04_P1.00mm_Horizontal" H 2650 4250 50  0001 C CNN
 F 3 "~" H 2650 4250 50  0001 C CNN
 	1    2650 4250
@@
 F 0 "U3" H 5550 7475 50  0000 C CNN
 F 1 "RIGHT_TB6612FNG" H 5550 7384 50  0000 C CNN
-F 2 "" H 5350 6950 50  0001 C CNN
+F 2 "Module:TB6612FNG" H 5350 6950 50  0001 C CNN
 F 3 "" H 5350 6950 50  0001 C CNN
 	1    5550 6950
@@
 F 0 "J4" H 7918 4117 50  0000 C CNN
 F 1 "Conn_VL53L0X" H 7918 4026 50  0000 C CNN
-F 2 "" H 8000 3700 50  0001 C CNN
+F 2 "Connector_PinHeader_1.00mm:PinHeader_1x06_P1.00mm_Horizontal" H 8000 3700 50  0001 C CNN
 F 3 "~" H 8000 3700 50  0001 C CNN
 	1    8000 3700
@@
 F 0 "J5" H 7918 4967 50  0000 C CNN
 F 1 "Conn_VL53L0X" H 7918 4876 50  0000 C CNN
-F 2 "" H 8000 4550 50  0001 C CNN
+F 2 "Connector_PinHeader_1.00mm:PinHeader_1x06_P1.00mm_Horizontal" H 8000 4550 50  0001 C CNN
 F 3 "~" H 8000 4550 50  0001 C CNN
 	1    8000 4550
@@
 F 0 "J6" H 7918 5817 50  0000 C CNN
 F 1 "Conn_VL53L0X" H 7918 5726 50  0000 C CNN
-F 2 "" H 8000 5400 50  0001 C CNN
+F 2 "Connector_PinHeader_1.00mm:PinHeader_1x06_P1.00mm_Horizontal" H 8000 5400 50  0001 C CNN
 F 3 "~" H 8000 5400 50  0001 C CNN
 	1    8000 5400
@@
 F 0 "J7" H 1868 7167 50  0000 C CNN
 F 1 "Conn_MOTOR_LEFT" H 1868 7076 50  0000 C CNN
-F 2 "" H 1950 6950 50  0001 C CNN
+F 2 "Connector_PinHeader_1.00mm:PinHeader_1x02_P1.00mm_Horizontal" H 1950 6950 50  0001 C CNN
 F 3 "~" H 1950 6950 50  0001 C CNN
 	1    1950 6950
@@
 F 0 "J8" H 4218 7367 50  0000 C CNN
 F 1 "Conn_MOTOR_RIGHT" H 4218 7276 50  0000 C CNN
-F 2 "" H 4300 7150 50  0001 C CNN
+F 2 "Connector_PinHeader_1.00mm:PinHeader_1x02_P1.00mm_Horizontal" H 4300 7150 50  0001 C CNN
 F 3 "~" H 4300 7150 50  0001 C CNN
 	1    4300 7150

Commit message: schematic v3 and PCB v2
Connections:
- net 5V_ARDUINO: now also J2.2 (Pin_2), J3.2 (Pin_2), J4.3 (Pin_3), J5.6 (Pin_6), J6.3 (Pin_3); no longer J2.1 (Pin_1), J3.1 (Pin_1), J4.1 (Pin_1), J5.1 (Pin_1), J6.1 (Pin_1)
- net ANALOG_LINE1: now also J2.3 (Pin_3); no longer J2.4 (Pin_4)
- net ANALOG_LINE2: now also J3.3 (Pin_3); no longer J3.4 (Pin_4)
- net BIT1_MOTOR_LEFT: now also A1.10 (D7); no longer A1.8 (D5)
- net BIT1_MOTOR_RIGHT: now also A1.15 (D12); no longer A1.10 (D7)
- net BIT2_MOTOR_LEFT: now also A1.11 (D8); no longer A1.9 (D6)
- net BIT2_MOTOR_RIGHT: now also A1.14 (D11); no longer A1.11 (D8)
- net DISTANCE_02: now also J5.1 (Pin_1); no longer J5.6 (Pin_6)
- net DISTANCE_03: now also A1.5 (D2); no longer A1.15 (D12)
- net GND: now also J2.1 (Pin_1), J3.1 (Pin_1), J4.4 (Pin_4), J5.3 (Pin_3), J6.4 (Pin_4); no longer J2.2 (Pin_2), J3.2 (Pin_2), J4.2 (Pin_2), J5.2 (Pin_2), J6.2 (Pin_2)
- net PWM_MOTOR_LEFT: now also A1.12 (D9); no longer A1.13 (D10)
- net PWM_MOTOR_RIGHT: now also A1.13 (D10); no longer A1.14 (D11)
- net SCL_VL53L0X: now also J4.2 (Pin_2), J5.5 (Pin_5), J6.2 (Pin_2); no longer J4.3 (Pin_3), J5.3 (Pin_3), J6.3 (Pin_3)
- net SDA_VL53L0X: now also J4.1 (Pin_1), J6.1 (Pin_1); no longer J4.4 (Pin_4), J6.4 (Pin_4)
- net SIGNAL_MICROSTART: now also A1.8 (D5); no longer A1.5 (D2)
- net STBY_TB6612FNG: now also A1.9 (D6); no longer A1.12 (D9)
- net at U3.6 (B02): now also J8.2 (Pin_2); no longer J8.1 (Pin_1)
- net at U3.7 (B01): now also J8.1 (Pin_1); no longer J8.2 (Pin_2)
- net at U4.4 (A01): now also J7.2 (Pin_2); no longer J7.1 (Pin_1)
- net at U4.5 (A02): now also J7.1 (Pin_1); no longer J7.2 (Pin_2)
Changed lines of the file:
@@
 Sheet 1 1
 Title "Vadeco"
-Date "2021-05-30"
-Rev "02"
+Date "2021-06-02"
+Rev "03"
 Comp "Robotech"
 Comment1 "Dev.: José Neto"
@@
 	-1   0    0    -1
 $EndComp
-Text GLabel 2850 4150 2    50   Input ~ 0
-5V_ARDUINO
-Text GLabel 2850 3500 2    50   Input ~ 0
-5V_ARDUINO
-Text GLabel 2850 3600 2    50   UnSpc ~ 0
-GND
-Text GLabel 2850 4250 2    50   UnSpc ~ 0
-GND
-Text GLabel 2850 4450 2    50   Output ~ 0
+Text GLabel 2850 4250 2    50   Input ~ 0
+5V_ARDUINO
+Text GLabel 2850 3600 2    50   Input ~ 0
+5V_ARDUINO
+Text GLabel 2850 3500 2    50   UnSpc ~ 0
+GND
+Text GLabel 2850 4150 2    50   UnSpc ~ 0
+GND
+Text GLabel 2850 4350 2    50   Output ~ 0
 ANALOG_LINE2
-Text GLabel 2850 3800 2    50   Output ~ 0
+Text GLabel 2850 3700 2    50   Output ~ 0
 ANALOG_LINE1
 $Comp
@@
 	-1   0    0    -1
 $EndComp
-Text GLabel 8200 3500 2    50   Input ~ 0
-5V_ARDUINO
-Text GLabel 8200 4350 2    50   Input ~ 0
-5V_ARDUINO
-Text GLabel 8200 3600 2    50   UnSpc ~ 0
-GND
-Text GLabel 8200 4450 2    50   UnSpc ~ 0
-GND
-Text GLabel 8200 3700 2    50   Input ~ 0
+Text GLabel 8200 4850 2    50   Input ~ 0
+5V_ARDUINO
+Text GLabel 8200 4550 2    50   UnSpc ~ 0
+GND
+Text GLabel 8200 4750 2    50   Input ~ 0
 SCL_VL53L0X
-Text GLabel 8200 4550 2    50   Input ~ 0
-SCL_VL53L0X
-Text GLabel 8200 3800 2    50   BiDi ~ 0
-SDA_VL53L0X
 Text GLabel 8200 4650 2    50   BiDi ~ 0
 SDA_VL53L0X
 NoConn ~ 8200 3900
-NoConn ~ 8200 4750
+NoConn ~ 8200 4450
 Text GLabel 8200 4000 2    50   Input ~ 0
 DISTANCE_01
@@
 $EndComp
 NoConn ~ 8200 5600
-Text GLabel 8200 4850 2    50   Input ~ 0
+Text GLabel 8200 4350 2    50   Input ~ 0
 DISTANCE_02
 Text GLabel 8200 5700 2    50   Input ~ 0
 DISTANCE_03
-Text GLabel 8200 5200 2    50   Input ~ 0
-5V_ARDUINO
-Text GLabel 8200 5300 2    50   UnSpc ~ 0
-GND
 Text GLabel 8200 5400 2    50   Input ~ 0
+5V_ARDUINO
+Text GLabel 8200 5500 2    50   UnSpc ~ 0
+GND
+Text GLabel 8200 5300 2    50   Input ~ 0
 SCL_VL53L0X
-Text GLabel 8200 5500 2    50   BiDi ~ 0
+Text GLabel 8200 5200 2    50   BiDi ~ 0
 SDA_VL53L0X
 Text GLabel 5150 6650 0    50   Input ~ 0
@@
 Text GLabel 6350 5200 2    50   Output ~ 0
 SCL_VL53L0X
-Text GLabel 5350 4300 0    50   Input ~ 0
+Text GLabel 5350 4600 0    50   Input ~ 0
 SIGNAL_MICROSTART
 Text GLabel 6350 4700 2    50   Input ~ 0
@@
 L Connector_Generic:Conn_01x02 J7
 U 1 1 60BCBAF1
-P 1950 6950
-F 0 "J7" H 1868 7167 50  0000 C CNN
-F 1 "Conn_MOTOR_LEFT" H 1868 7076 50  0000 C CNN
-F 2 "Connector_PinHeader_1.00mm:PinHeader_1x02_P1.00mm_Horizontal" H 1950 6950 50  0001 C CNN
-F 3 "~" H 1950 6950 50  0001 C CNN
-	1    1950 6950
-	-1   0    0    -1
+P 1950 7050
+F 0 "J7" H 1868 7267 50  0000 C CNN
+F 1 "Conn_MOTOR_LEFT" H 1868 7176 50  0000 C CNN
+F 2 "Connector_PinHeader_1.00mm:PinHeader_1x02_P1.00mm_Horizontal" H 1950 7050 50  0001 C CNN
+F 3 "~" H 1950 7050 50  0001 C CNN
+	1    1950 7050
+	-1   0    0    1
 $EndComp
 Wire Wire Line
@@
 L Connector_Generic:Conn_01x02 J8
 U 1 1 60BCDDB0
-P 4300 7150
-F 0 "J8" H 4218 7367 50  0000 C CNN
-F 1 "Conn_MOTOR_RIGHT" H 4218 7276 50  0000 C CNN
-F 2 "Connector_PinHeader_1.00mm:PinHeader_1x02_P1.00mm_Horizontal" H 4300 7150 50  0001 C CNN
-F 3 "~" H 4300 7150 50  0001 C CNN
-	1    4300 7150
-	-1   0    0    -1
+P 4300 7250
+F 0 "J8" H 4218 7467 50  0000 C CNN
+F 1 "Conn_MOTOR_RIGHT" H 4218 7376 50  0000 C CNN
+F 2 "Connector_PinHeader_1.00mm:PinHeader_1x02_P1.00mm_Horizontal" H 4300 7250 50  0001 C CNN
+F 3 "~" H 4300 7250 50  0001 C CNN
+	1    4300 7250
+	-1   0    0    1
 $EndComp
 Wire Wire Line
@@
 Text GLabel 5950 7250 2    50   Input ~ 0
 PWM_MOTOR_RIGHT
+Text GLabel 5350 5000 0    50   Output ~ 0
+PWM_MOTOR_LEFT
 Text GLabel 5350 5100 0    50   Output ~ 0
-PWM_MOTOR_LEFT
-Text GLabel 5350 5200 0    50   Output ~ 0
 PWM_MOTOR_RIGHT
 Text GLabel 3600 6750 2    50   Input ~ 0
@@
 Text GLabel 5950 7150 2    50   Input ~ 0
 BIT2_MOTOR_RIGHT
-Text GLabel 5350 4600 0    50   Output ~ 0
+Text GLabel 5350 4800 0    50   Output ~ 0
 BIT1_MOTOR_LEFT
+Text GLabel 5350 4900 0    50   Output ~ 0
+BIT2_MOTOR_LEFT
+Text GLabel 5350 5300 0    50   Output ~ 0
+BIT1_MOTOR_RIGHT
+Text GLabel 5350 5200 0    50   Output ~ 0
+BIT2_MOTOR_RIGHT
 Text GLabel 5350 4700 0    50   Output ~ 0
-BIT2_MOTOR_LEFT
-Text GLabel 5350 4800 0    50   Output ~ 0
-BIT1_MOTOR_RIGHT
-Text GLabel 5350 4900 0    50   Output ~ 0
-BIT2_MOTOR_RIGHT
-Text GLabel 5350 5000 0    50   Output ~ 0
 STBY_TB6612FNG
 Text GLabel 3600 6950 2    50   Input ~ 0
@@
 Text GLabel 5950 6950 2    50   Input ~ 0
 STBY_TB6612FNG
-NoConn ~ 2850 3700
-NoConn ~ 2850 4350
+NoConn ~ 2850 3800
+NoConn ~ 2850 4450
 Text GLabel 5350 4400 0    50   Input ~ 0
 DISTANCE_01
 Text GLabel 5350 4500 0    50   Input ~ 0
 DISTANCE_02
-Text GLabel 5350 5300 0    50   Input ~ 0
+Text GLabel 5350 4300 0    50   Input ~ 0
 DISTANCE_03
 Wire Notes Line style solid
@@
 	7100 2400 7100 3000
 NoConn ~ 5350 5400
+Text GLabel 8200 3800 2    50   UnSpc ~ 0
+GND
+Text GLabel 8200 3700 2    50   Input ~ 0
+5V_ARDUINO
+Text GLabel 8200 3600 2    50   Input ~ 0
+SCL_VL53L0X
+Text GLabel 8200 3500 2    50   BiDi ~ 0
+SDA_VL53L0X
 $EndSCHEMATC
